File: geiger.brd (EAGLE design)
At the start: 160 x 100 mm, 17 parts, among them IC1 MC34063A, Q1 IRF840, Q2 2N3906, Q3 2N3906, X1 22-23-2021, X2 22-23-2021

Commit message: fixes
Parts:
- added C4: 100n, rcl:C025-025X050
- added R5: 20k, rcl:0204/7
- C1: value (none) -> 4.7n
- C3: value 100u/1kV -> 22n/1kV
- R1: value 0.05 -> 22
- R3: value 31k -> 10k
Connections:
- new net N$4: R3.1, R5.2
- net +5V: now also C4.1
- net GND: now also C4.2, R5.1; no longer R3.1
Routing:
- net N$4: track 0.00 -> 3.81 mm
- net +5V: track 21.3 -> 24.9 mm
Changed lines of the file:
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@@
 </autorouter>
 <elements>
-<element name="C1" library="rcl" library_urn="urn:adsk.eagle:library:334" package="C025-025X050" package3d_urn="urn:adsk.eagle:package:23629/2" value="" x="73.66" y="33.02" rot="R90"/>
+<element name="C1" library="rcl" library_urn="urn:adsk.eagle:library:334" package="C025-025X050" package3d_urn="urn:adsk.eagle:package:23629/2" value="4.7n" x="73.66" y="33.02" rot="R90"/>
 <element name="C2" library="rcl" library_urn="urn:adsk.eagle:library:334" package="C025-025X050" package3d_urn="urn:adsk.eagle:package:23629/2" value="100n" x="67.31" y="82.55" rot="R180"/>
 <element name="D1" library="diode" library_urn="urn:adsk.eagle:library:210" package="DO35-10" package3d_urn="urn:adsk.eagle:package:43344/2" value="1N4148DO35-10" x="66.04" y="36.83" rot="R90"/>
@@
 <element name="Q2" library="transistor-pnp" library_urn="urn:adsk.eagle:library:399" package="TO92" package3d_urn="urn:adsk.eagle:package:29211/2" value="2N3906" x="53.34" y="41.91" rot="R270"/>
 <element name="Q3" library="transistor-pnp" library_urn="urn:adsk.eagle:library:399" package="TO92" package3d_urn="urn:adsk.eagle:package:29211/2" value="2N3906" x="73.66" y="41.91" rot="R90"/>
-<element name="R1" library="rcl" library_urn="urn:adsk.eagle:library:334" package="0204/7" package3d_urn="urn:adsk.eagle:package:23498/1" value="0.05" x="52.07" y="69.85"/>
+<element name="R1" library="rcl" library_urn="urn:adsk.eagle:library:334" package="0204/7" package3d_urn="urn:adsk.eagle:package:23498/1" value="22" x="52.07" y="69.85"/>
 <element name="R2" library="rcl" library_urn="urn:adsk.eagle:library:334" package="0204/7" package3d_urn="urn:adsk.eagle:package:23498/1" value="10k" x="62.23" y="38.1" rot="R90"/>
-<element name="R3" library="rcl" library_urn="urn:adsk.eagle:library:334" package="0204/7" package3d_urn="urn:adsk.eagle:package:23498/1" value="31k" x="72.39" y="77.47" rot="R180"/>
+<element name="R3" library="rcl" library_urn="urn:adsk.eagle:library:334" package="0204/7" package3d_urn="urn:adsk.eagle:package:23498/1" value="10k" x="72.39" y="77.47" rot="R180"/>
 <element name="R4" library="rcl" library_urn="urn:adsk.eagle:library:334" package="0204/7" package3d_urn="urn:adsk.eagle:package:23498/1" value="10M" x="52.07" y="77.47" rot="R180"/>
 <element name="X1" library="con-molex" library_urn="urn:adsk.eagle:library:165" package="22-23-2021" value="22-23-2021" x="60.96" y="71.12" rot="R90">
@@
 <attribute name="OC_NEWARK" value="25C3832" x="46.99" y="83.82" size="1.778" layer="27" display="off"/>
 </element>
-<element name="C3" library="rcl" library_urn="urn:adsk.eagle:library:334" package="C050-050X075" package3d_urn="urn:adsk.eagle:package:23665/1" value="100u/1kV" x="39.37" y="83.82"/>
+<element name="C3" library="rcl" library_urn="urn:adsk.eagle:library:334" package="C050-050X075" package3d_urn="urn:adsk.eagle:package:23665/1" value="22n/1kV" x="39.37" y="83.82"/>
+<element name="R5" library="rcl" library_urn="urn:adsk.eagle:library:334" package="0204/7" package3d_urn="urn:adsk.eagle:package:23498/1" value="20k" x="76.2" y="69.85" rot="R90"/>
+<element name="C4" library="rcl" library_urn="urn:adsk.eagle:library:334" package="C025-025X050" package3d_urn="urn:adsk.eagle:package:23629/2" value="100n" x="60.96" y="63.5" rot="R180"/>
 </elements>
 <signals>
@@
 <contactref element="Q3" pad="1"/>
 <contactref element="IC1" pad="4"/>
-<contactref element="R3" pad="1"/>
 <contactref element="C2" pad="2"/>
 <contactref element="Q1" pad="3"/>
@@
 </polygon>
 <contactref element="C3" pad="2"/>
+<contactref element="R5" pad="1"/>
+<contactref element="C4" pad="2"/>
 </signal>
 <signal name="N$5">
@@
 <wire x1="60.96" y1="69.9516" x2="60.96" y2="69.85" width="0.1524" layer="16"/>
 <wire x1="65.9892" y1="64.77" x2="65.9892" y2="55.9308" width="0.1524" layer="16"/>
-<wire x1="60.96" y1="69.7992" x2="65.9892" y2="64.77" width="0.1524" layer="16"/>
+<wire x1="60.96" y1="69.7992" x2="64.77" y2="65.9892" width="0.1524" layer="16"/>
+<wire x1="64.77" y1="65.9892" x2="65.9892" y2="64.77" width="0.1524" layer="16"/>
 <wire x1="65.9892" y1="55.9308" x2="66.04" y2="55.88" width="0.1524" layer="16"/>
 <wire x1="60.96" y1="69.7992" x2="60.96" y2="69.85" width="0.1524" layer="16"/>
+<contactref element="C4" pad="1"/>
+<wire x1="64.77" y1="65.9892" x2="62.3316" y2="63.5508" width="0.1524" layer="16"/>
+<wire x1="62.3316" y1="63.5508" x2="62.23" y2="63.5" width="0.1524" layer="16"/>
 </signal>
 <signal name="N$3">
@@
 <wire x1="62.3316" y1="41.91" x2="62.23" y2="41.91" width="0.1524" layer="16"/>
 </signal>
+<signal name="N$4">
+<contactref element="R3" pad="1"/>
+<contactref element="R5" pad="2"/>
+<wire x1="76.2" y1="77.47" x2="76.2" y2="73.66" width="0.1524" layer="16"/>
+</signal>
 </signals>

Commit message: beeping
Parts:
- added C5: 330u/630v, rcl:C050-050X075
- added C6: 100u, rcl:C025-025X050
- added C7: 330p, rcl:C025-025X050
- added C8: 10n, rcl:C025-025X050
- added C9: 47n, rcl:C025-025X050
- added IC2: NE555, st-microelectronics:DIL-08
- added Q4, Q5: 2N3904, transistor-npn:TO92
- added R10: 10k, rcl:0204/7
- added R11: 1M, rcl:0204/7
- added R12, R6: 10, rcl:0204/7
- added R13: 0, rcl:0204/7
- added R7: 300k, rcl:0204/7
- added R8: 5M, rcl:0204/7
- added R9: 100, rcl:0204/7
- added SP1: KSS1201, buzzer:KSS1201
- R1: value 22 -> 0
- moved X2 36.9 mm to (10.2, 85.1)
- moved C2 27.7 mm to (74.9, 55.9), turned to 0 degrees
- moved R5 21.6 mm to (61.0, 85.1), turned to 0 degrees
- moved C3 11.7 mm to (31.8, 74.9), turned to 270 degrees
- moved L1 9.92 mm to (44.5, 62.2)
- moved C1 9.67 mm to (77.5, 41.9)
- moved R3 5.39 mm to (68.6, 81.3), turned to 270 degrees
- moved D2 5.39 mm to (39.4, 73.7), turned to 270 degrees
- moved C4 2.54 mm to (58.4, 63.5), turned to 270 degrees
- moved X1 2.54 mm to (58.4, 71.1)
- moved R1 1.27 mm to (50.8, 69.8), turned to 90 degrees
Connections:
- removed net +5V: C4.1, IC1.6, R1.2, X1.1
- new net N$10: C7.1, Q5.2, R7.2, X2.1
- new net N$12: R8.2, X2.2
- new net N$13: IC2.2, Q5.1, R10.1
- new net N$14: C8.1, IC2.5
- new net N$15: IC2.3, R9.1
- new net N$16: Q4.2, R9.2
- new net N$17: Q4.1, SP1.-
- new net N$18: C9.1, IC2.6, IC2.7, R11.1
- new net N$19: R12.1, SP1.+
- new net N$7: IC2.4, IC2.8, R10.2, R11.2, R12.2, R13.1
- new net N$9: Q1.1, R6.2
- new net VCC: C4.1, C6.1, IC1.6, R1.2, R13.2, X1.1
- net GND: now also C5.2, C6.2, C7.2, C8.2, C9.2, IC2.1, Q4.3, Q5.3, R7.1; no longer X2.1
- net N$6: now also R6.1; no longer Q1.1
- net N$8: now also C5.1, R8.1; no longer X2.2
Routing:
- net N$7: track 0.00 -> 146.2 mm
- net VCC: track 0.00 -> 32.8 mm
- net N$13: track 0.00 -> 31.3 mm
- net +5V: track 24.9 -> 0.00 mm
- net N$17: track 0.00 -> 17.1 mm
- net N$10: track 0.00 -> 16.2 mm
- net N$19: track 0.00 -> 12.4 mm
- net N$8: track 22.8 -> 33.3 mm
- net N$18: track 0.00 -> 10.4 mm
- net N$3: track 36.7 -> 27.7 mm
- net N$16: track 0.00 -> 8.54 mm
- net N$9: track 0.00 -> 8.45 mm
- net N$5: track 33.3 -> 26.9 mm
- net N$6: track 17.9 -> 11.6 mm
- net N$15: track 0.00 -> 5.15 mm
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Other:
- board size 160 x 100 mm -> 87.6 x 75.9 mm
