File: geiger.sch (EAGLE design)
At the start: 17 parts, among them IC1 MC34063A, Q1 IRF840, Q2 2N3906, Q3 2N3906, X1 22-23-2021, X2 22-23-2021

Commit message: fixes
Parts:
- added C4: 100n, rcl:C-EU025-025X050
- added R5: 20k, rcl:R-EU_0204/7
- C1: value (none) -> 4.7n
- C3: value 100u/1kV -> 22n/1kV
- R1: value 0.05 -> 22
- R3: value 31k -> 10k
Connections:
- new net N$4: R3.1, R5.2
- net +5V: now also C4.1
- net GND: now also C4.2, R5.1; no longer R3.1
Other:
- moved on the sheet: X1-1, X1-2
Changed lines of the file:
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@@
 <part name="IC1" library="ic-package" library_urn="urn:adsk.eagle:library:239" deviceset="DIL8" device="" package3d_urn="urn:adsk.eagle:package:14440/1" value="MC34063A"/>
 <part name="D1" library="diode" library_urn="urn:adsk.eagle:library:210" deviceset="1N4148" device="DO35-10" package3d_urn="urn:adsk.eagle:package:43344/2"/>
-<part name="C1" library="rcl" library_urn="urn:adsk.eagle:library:334" deviceset="C-EU" device="025-025X050" package3d_urn="urn:adsk.eagle:package:23629/2"/>
+<part name="C1" library="rcl" library_urn="urn:adsk.eagle:library:334" deviceset="C-EU" device="025-025X050" package3d_urn="urn:adsk.eagle:package:23629/2" value="4.7n"/>
 <part name="SUPPLY1" library="supply2" library_urn="urn:adsk.eagle:library:372" deviceset="GND" device=""/>
 <part name="SUPPLY2" library="supply2" library_urn="urn:adsk.eagle:library:372" deviceset="GND" device=""/>
-<part name="R1" library="rcl" library_urn="urn:adsk.eagle:library:334" deviceset="R-EU_" device="0204/7" package3d_urn="urn:adsk.eagle:package:23498/1" value="0.05"/>
-<part name="R3" library="rcl" library_urn="urn:adsk.eagle:library:334" deviceset="R-EU_" device="0204/7" package3d_urn="urn:adsk.eagle:package:23498/1" value="31k"/>
+<part name="R1" library="rcl" library_urn="urn:adsk.eagle:library:334" deviceset="R-EU_" device="0204/7" package3d_urn="urn:adsk.eagle:package:23498/1" value="22"/>
+<part name="R3" library="rcl" library_urn="urn:adsk.eagle:library:334" deviceset="R-EU_" device="0204/7" package3d_urn="urn:adsk.eagle:package:23498/1" value="10k"/>
 <part name="R4" library="rcl" library_urn="urn:adsk.eagle:library:334" deviceset="R-EU_" device="0204/7" package3d_urn="urn:adsk.eagle:package:23498/1" value="10M"/>
 <part name="SUPPLY3" library="supply2" library_urn="urn:adsk.eagle:library:372" deviceset="GND" device=""/>
@@
 <part name="SUPPLY8" library="supply2" library_urn="urn:adsk.eagle:library:372" deviceset="GND" device=""/>
 <part name="SUPPLY9" library="supply2" library_urn="urn:adsk.eagle:library:372" deviceset="GND" device=""/>
-<part name="C3" library="rcl" library_urn="urn:adsk.eagle:library:334" deviceset="C-EU" device="050-050X075" package3d_urn="urn:adsk.eagle:package:23665/1" value="100u/1kV"/>
+<part name="C3" library="rcl" library_urn="urn:adsk.eagle:library:334" deviceset="C-EU" device="050-050X075" package3d_urn="urn:adsk.eagle:package:23665/1" value="22n/1kV"/>
 <part name="SUPPLY10" library="supply2" library_urn="urn:adsk.eagle:library:372" deviceset="GND" device=""/>
+<part name="R5" library="rcl" library_urn="urn:adsk.eagle:library:334" deviceset="R-EU_" device="0204/7" package3d_urn="urn:adsk.eagle:package:23498/1" value="20k"/>
+<part name="C4" library="rcl" library_urn="urn:adsk.eagle:library:334" deviceset="C-EU" device="025-025X050" package3d_urn="urn:adsk.eagle:package:23629/2" value="100n"/>
+<part name="SUPPLY11" library="supply2" library_urn="urn:adsk.eagle:library:372" deviceset="GND" device=""/>
 </parts>
 <sheets>
@@
 <instance part="R3" gate="G$1" x="7.62" y="45.72" rot="R90"/>
 <instance part="R4" gate="G$1" x="7.62" y="55.88" rot="R90"/>
-<instance part="SUPPLY3" gate="GND" x="7.62" y="38.1"/>
-<instance part="P+1" gate="1" x="71.12" y="73.66"/>
+<instance part="SUPPLY3" gate="GND" x="2.54" y="27.94"/>
+<instance part="P+1" gate="1" x="73.66" y="73.66"/>
 <instance part="C2" gate="G$1" x="-7.62" y="48.26"/>
 <instance part="SUPPLY5" gate="GND" x="-7.62" y="38.1"/>
@@
 <instance part="Q3" gate="G$1" x="63.5" y="20.32"/>
 <instance part="SUPPLY7" gate="GND" x="40.64" y="-5.08"/>
-<instance part="X1" gate="-1" x="86.36" y="66.04"/>
-<instance part="X1" gate="-2" x="86.36" y="63.5"/>
+<instance part="X1" gate="-1" x="91.44" y="66.04"/>
+<instance part="X1" gate="-2" x="91.44" y="63.5"/>
 <instance part="X2" gate="-1" x="-22.86" y="63.5" rot="R180"/>
 <instance part="X2" gate="-2" x="-22.86" y="66.04" rot="R180"/>
 <instance part="SUPPLY8" gate="GND" x="-17.78" y="60.96"/>
-<instance part="SUPPLY9" gate="GND" x="81.28" y="60.96"/>
+<instance part="SUPPLY9" gate="GND" x="88.9" y="60.96"/>
 <instance part="C3" gate="G$1" x="-7.62" y="63.5"/>
 <instance part="SUPPLY10" gate="GND" x="-7.62" y="55.88"/>
+<instance part="R5" gate="G$1" x="7.62" y="35.56" rot="R90"/>
+<instance part="C4" gate="G$1" x="73.66" y="63.5"/>
+<instance part="SUPPLY11" gate="GND" x="73.66" y="55.88"/>
 </instances>
 <busses>
@@
 </segment>
 <segment>
-<pinref part="R3" gate="G$1" pin="1"/>
-<pinref part="SUPPLY3" gate="GND" pin="GND"/>
-</segment>
-<segment>
 <pinref part="C2" gate="G$1" pin="2"/>
 <pinref part="SUPPLY5" gate="GND" pin="GND"/>
@@
 <pinref part="X1" gate="-2" pin="S"/>
 <pinref part="SUPPLY9" gate="GND" pin="GND"/>
-<wire x1="81.28" y1="63.5" x2="83.82" y2="63.5" width="0.1524" layer="91"/>
 </segment>
 <segment>
 <pinref part="C3" gate="G$1" pin="2"/>
 <pinref part="SUPPLY10" gate="GND" pin="GND"/>
+</segment>
+<segment>
+<pinref part="R5" gate="G$1" pin="1"/>
+<pinref part="SUPPLY3" gate="GND" pin="GND"/>
+<wire x1="2.54" y1="30.48" x2="7.62" y2="30.48" width="0.1524" layer="91"/>
+</segment>
+<segment>
+<pinref part="SUPPLY11" gate="GND" pin="GND"/>
+<pinref part="C4" gate="G$1" pin="2"/>
 </segment>
 </net>
@@
 <pinref part="R1" gate="G$1" pin="2"/>
 <pinref part="P+1" gate="1" pin="+5V"/>
-<wire x1="71.12" y1="71.12" x2="71.12" y2="66.04" width="0.1524" layer="91"/>
+<wire x1="73.66" y1="71.12" x2="73.66" y2="66.04" width="0.1524" layer="91"/>
 <pinref part="IC1" gate="G$1" pin="6"/>
-<wire x1="60.96" y1="55.88" x2="71.12" y2="66.04" width="0.1524" layer="91"/>
-<junction x="71.12" y="66.04"/>
+<wire x1="60.96" y1="55.88" x2="73.66" y2="66.04" width="0.1524" layer="91"/>
+<junction x="73.66" y="66.04"/>
 <pinref part="X1" gate="-1" pin="S"/>
-<wire x1="71.12" y1="66.04" x2="83.82" y2="66.04" width="0.1524" layer="91"/>
+<wire x1="73.66" y1="66.04" x2="88.9" y2="66.04" width="0.1524" layer="91"/>
+<pinref part="C4" gate="G$1" pin="1"/>
+<wire x1="73.66" y1="66.04" x2="71.12" y2="66.04" width="0.1524" layer="91"/>
 </segment>
 </net>
@@
 </segment>
 </net>
+<net name="N$4" class="0">
+<segment>
+<pinref part="R3" gate="G$1" pin="1"/>
+<pinref part="R5" gate="G$1" pin="2"/>
+</segment>
+</net>

Commit message: beeping
Parts:
- added C5: 330u/630v, rcl:C-EU050-050X075
- added C6: 100u, rcl:C-EU025-025X050
- added C7: 330p, rcl:C-EU025-025X050
- added C8: 10n, rcl:C-EU025-025X050
- added C9: 47n, rcl:C-EU025-025X050
- added IC2: NE555, st-microelectronics:NE555
- added Q4, Q5: 2N3904, transistor-npn:2N3904
- added R10: 10k, rcl:R-EU_0204/7
- added R11: 1M, rcl:R-EU_0204/7
- added R12, R6: 10, rcl:R-EU_0204/7
- added R13: 0, rcl:R-EU_0204/7
- added R7: 300k, rcl:R-EU_0204/7
- added R8: 5M, rcl:R-EU_0204/7
- added R9: 100, rcl:R-EU_0204/7
- added SP1: KSS1201, buzzer:KSS1201
- R1: value 22 -> 0
Connections:
- removed net +5V: C4.1, IC1.6, R1.2, X1-1.S
- new net N$10: C7.1, Q5.B, R7.2, X2-1.S
- new net N$12: R8.2, X2-2.S
- new net N$13: IC2.TRI, Q5.C, R10.1
- new net N$14: C8.1, IC2.CON
- new net N$15: IC2.OUT, R9.1
- new net N$16: Q4.B, R9.2
- new net N$17: Q4.C, SP1.2
- new net N$18: C9.1, IC2.DIS, IC2.TRE, R11.1
- new net N$19: R12.1, SP1.1
- new net N$7: IC2./RES, IC2.VCC+, R10.2, R11.2, R12.2, R13.1
- new net N$9: Q1.G, R6.2
- new net VCC: C4.1, C6.1, IC1.6, R1.2, R13.2, X1-1.S
- net GND: now also C5.2, C6.2, C7.2, C8.2, C9.2, IC2.GND, Q4.E, Q5.E, R7.1; no longer X2-1.S
- net N$6: now also R6.1; no longer Q1.G
- net N$8: now also C5.1, R8.1; no longer X2-2.S
Other:
- note added: "9v - 12v"
- note added: "DANGER: 400 VOLTS !"
- note added: "MC34063 Application Note 920 Ratio Extender Circuit"
- note added: "STS-5 400v"
- moved on the sheet: C1, C2, C3, C4, D2, D3, R4, R5, X1-1, X1-2, X2-1, X2-2
